File: Projects/NerveDetector/Guille/Byaxon_2D_V1/Byaxon_2D_V1.kicad_sch (KiCad schematic)
At the start: 74 parts, among them U1 TL074

Commit message: Solved problem with footprint libraries missing
Parts:
- removed H1, H2, H3: MountingHole_Pad, Library_Acid_etch_limitations:MountingHole_2.1mm_Acid_Etch_Limitations, symbol Mechanical:MountingHole_Pad
- R1, R2, R3: footprint SamacSys_Parts:ERJ1T__2512_ -> Samac_sys:ERJ1T__2512_
- R10, R11, R12, R9: footprint SamacSys_Parts:RESC1608X60N -> Samac_sys:RESC1608X60N
- R14, R20: footprint SamacSys_Parts:RESC1608X55N -> Samac_sys:RESC3016X65N; Height 0.55 -> 0.65; Manufacturer_Name Arcol -> Stackpole Electronics, Inc.; Manufacturer_Part_Number APC0603T10K0Z -> RNCF1206TKY200R; Mouser Part Number 284-APC0603T10K0Z -> 708-RNCF1206TKY200R; Mouser Price/Stock https://www.mouser.co.uk/ProductDetail/ARCOL-Ohmite/APC0603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 -> (none)
- R26, R4, R5: footprint RESC3016X65N -> Samac_sys:RESC3016X65N; Mouser Part Number (none) -> 708-RNCF1206TKY200R

Commit message: Layed out bigger edge cut, added jumper to Voss
Parts:
- added J11, J12, J13, J14: ~, Connector_Pin:Pin_D0.7mm_L6.5mm_W1.8mm_FlatFork, symbol Connector_Generic:Conn_01x01
Connections:
- net Earth: now also J12.1 (Pin_1)
- net at R6.2, U1.1: now also J13.1 (Pin_1); no longer INA217_1.5 (Ref)
- new net: INA217_1.5 (Ref), J11.1 (Pin_1), J14.1 (Pin_1)
Other:
- moved on the sheet: R10, R28, R6, R9, U1A, VR1

Commit message: Changed jumpers + some layout
Parts:
- removed J11: ~, Connector_Pin:Pin_D0.7mm_L6.5mm_W1.8mm_FlatFork, symbol Connector_Generic:Conn_01x01
- added J15, J16, J18: ~, Connector_Pin:Pin_D0.7mm_L6.5mm_W1.8mm_FlatFork, symbol Connector_Generic:Conn_01x01
Connections:
- net Earth: now also J18.1 (Pin_1)
- net at R7.2, U1.7: now also J15.1 (Pin_1); no longer INA217_6.5 (Ref)
- new net: INA217_6.5 (Ref), J16.1 (Pin_1)
Other:
- note added: "Conectar un jumper o el otro según se quiera corregir V offset o no. Asegurar baja impedancia a tierra!"
- moved on the sheet: J12, J13, J14, R11, R12, R7, R8, U1B, VR2

Commit message: Final commit of the day - Some layout
Changed lines of the file:
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@@
   (symbol (lib_id "Device:R") (at 92.71 111.125 0) (unit 1)
     (in_bom yes) (on_board yes) (dnp no)
-    (property "Reference" "R10" (at 90.17 110.474 0)
+    (property "Reference" "R10" (at 89.535 110.49 0)
       (effects (font (size 1.27 1.27)))
     )

Commit message: Added mounting holes
Parts:
- added H1, H2, H3: MountingHole, MountingHole:MountingHole_3.2mm_M3, symbol Mechanical:MountingHole
- added H4: MountingHole_Pad, MountingHole:MountingHole_3.2mm_M3_DIN965_Pad, symbol Mechanical:MountingHole_Pad
Connections:
- net Earth: now also H4.1
Other:
- note added: "La carcasa se ata solo por un punto a tierra para evitar lazos de tierra."
Changed lines of the file:
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@@
     (stroke (width 0) (type default))
   )
+  (wire (pts (xy 391.16 60.96) (xy 391.16 62.23))
+    (stroke (width 0) (type default))
+  )
   (wire (pts (xy 57.15 213.995) (xy 58.42 213.995))
     (stroke (width 0.15) (type default))
@@
     (stroke (width 0) (type default))
   )
+  (rectangle (start 367.03 38.735) (end 402.59 78.105)
+    (stroke (width 0) (type default))
+    (fill (type none))
+  )
   (text_box "Gradiometer"
     (at 17.145 18.415 0) (size 22.86 5.08)
@@
     (effects (font (size 1.27 1.27)) (justify left bottom))
   )
+  (text "La carcasa se ata solo por un\npunto a tierra para evitar\nlazos de tierra."
+    (at 370.205 75.565 0)
+    (effects (font (size 1.27 1.27)) (justify left bottom))
+  )
   (text "Conectores through hole\npor si hay que cambiar resistencias"
     (at 100.33 59.69 0)
@@
     )
   )
+  (symbol (lib_id "power:Earth") (at 391.16 62.23 0) (unit 1)
+    (in_bom yes) (on_board yes) (dnp no) (fields_autoplaced)
+    (property "Reference" "#PWR016" (at 391.16 68.58 0)
+      (effects (font (size 1.27 1.27)) hide)
+    )
+    (property "Value" "Earth" (at 391.16 66.04 0)
+      (effects (font (size 1.27 1.27)) hide)
+    )
+    (property "Footprint" "" (at 391.16 62.23 0)
+      (effects (font (size 1.27 1.27)) hide)
+    )
+    (property "Datasheet" "~" (at 391.16 62.23 0)
+      (effects (font (size 1.27 1.27)) hide)
+    )
+    (pin "1")
+    (instances
+      (project "Byaxon_2D_V1"
+        (path "/eae49fa2-9ce6-4e5d-b671-c7c5bff76f9e"
+          (reference "#PWR016") (unit 1)
+        )
+      )
+    )
+  )
   (symbol (lib_id "power:Earth") (at 173.99 100.965 0) (unit 1)
     (in_bom yes) (on_board yes) (dnp no) (fields_autoplaced)
@@
     )
   )
+  (symbol (lib_id "Mechanical:MountingHole") (at 375.92 45.085 0) (unit 1)
+    (in_bom yes) (on_board yes) (dnp no)
+    (property "Reference" "H1" (at 374.65 41.91 0)
+      (effects (font (size 1.27 1.27)) (justify left))
+    )
+    (property "Value" "MountingHole" (at 370.205 48.26 0)
+      (effects (font (size 1.27 1.27)) (justify left))
+    )
+    (property "Footprint" "MountingHole:MountingHole_3.2mm_M3" (at 375.92 45.085 0)
+      (effects (font (size 1.27 1.27)) hide)
+    )
+    (property "Datasheet" "~" (at 375.92 45.085 0)
+      (effects (font (size 1.27 1.27)) hide)
+    )
+    (instances
+      (project "Byaxon_2D_V1"
+        (path "/eae49fa2-9ce6-4e5d-b671-c7c5bff76f9e"
+          (reference "H1") (unit 1)
+        )
+      )
+    )
+  )
   (symbol (lib_id "Connector_Generic:Conn_01x01") (at 170.18 90.805 0) (unit 1)
     (in_bom yes) (on_board yes) (dnp no)
@@
     )
   )
+  (symbol (lib_id "Mechanical:MountingHole_Pad") (at 391.16 58.42 0) (unit 1)
+    (in_bom yes) (on_board yes) (dnp no)
+    (property "Reference" "H4" (at 389.89 53.975 0)
+      (effects (font (size 1.27 1.27)) (justify left))
+    )
+    (property "Value" "MountingHole_Pad" (at 382.27 66.675 0)
+      (effects (font (size 1.27 1.27)) (justify left))
+    )
+    (property "Footprint" "MountingHole:MountingHole_3.2mm_M3_DIN965_Pad" (at 391.16 58.42 0)
+      (effects (font (size 1.27 1.27)) hide)
+    )
+    (property "Datasheet" "~" (at 391.16 58.42 0)
+      (effects (font (size 1.27 1.27)) hide)
+    )
+    (pin "1")
+    (instances
+      (project "Byaxon_2D_V1"
+        (path "/eae49fa2-9ce6-4e5d-b671-c7c5bff76f9e"
+          (reference "H4") (unit 1)
+        )
+      )
+    )
+  )
   (symbol (lib_id "Connector:Screw_Terminal_01x03") (at 339.725 86.995 180) (unit 1)
     (in_bom yes) (on_board yes) (dnp no)
@@
     )
   )
+  (symbol (lib_id "Mechanical:MountingHole") (at 375.92 57.15 0) (unit 1)
+    (in_bom yes) (on_board yes) (dnp no)
+    (property "Reference" "H3" (at 374.65 53.975 0)
+      (effects (font (size 1.27 1.27)) (justify left))
+    )
+    (property "Value" "MountingHole" (at 370.205 60.325 0)
+      (effects (font (size 1.27 1.27)) (justify left))
+    )
+    (property "Footprint" "MountingHole:MountingHole_3.2mm_M3" (at 375.92 57.15 0)
+      (effects (font (size 1.27 1.27)) hide)
+    )
+    (property "Datasheet" "~" (at 375.92 57.15 0)
+      (effects (font (size 1.27 1.27)) hide)
+    )
+    (instances
+      (project "Byaxon_2D_V1"
+        (path "/eae49fa2-9ce6-4e5d-b671-c7c5bff76f9e"
+          (reference "H3") (unit 1)
+        )
+      )
+    )
+  )
   (symbol (lib_id "Device:R") (at 65.405 144.145 90) (unit 1)
     (in_bom yes) (on_board yes) (dnp no)
@@
         )
       )
+    )
+  )
+  (symbol (lib_id "Mechanical:MountingHole") (at 391.16 45.085 0) (unit 1)
+    (in_bom yes) (on_board yes) (dnp no)
+    (property "Reference" "H2" (at 389.89 41.91 0)
+      (effects (font (size 1.27 1.27)) (justify left))
+    )
+    (property "Value" "MountingHole" (at 385.445 48.26 0)
+      (effects (font (size 1.27 1.27)) (justify left))
+    )
+    (property "Footprint" "MountingHole:MountingHole_3.2mm_M3" (at 391.16 45.085 0)
+      (effects (font (size 1.27 1.27)) hide)
+    )
+    (property "Datasheet" "~" (at 391.16 45.085 0)
+      (effects (font (size 1.27 1.27)) hide)
+    )
+    (instances
+      (project "Byaxon_2D_V1"
+        (path "/eae49fa2-9ce6-4e5d-b671-c7c5bff76f9e"
+          (reference "H2") (unit 1)
+        )
+      )
